File: 808_Kick.brd (EAGLE design)
At the start: 61.9 x 39.4 mm, 8 parts, among them IC1 TL072P, Q1 BC546A, Q2 BC546A, Q3 BC546A, Q4 BC546A, Q5 BC546A, Q6 BC556

Commit message: Updated
Parts:
- added C1, C10, C11, C12, C13, C14, C8, C9: (no value), capacitor-wima:C2.5-2
- added C2, C3, C4, C5, C6, C7: (no value), rcl:E2-5
- added D2, D3: 1N4148DO35-7, diode:DO35-7
- IC1: value TL072P -> TL072D; device linear:DIL08 -> linear:SO08
- Q1, Q2, Q3, Q5: value BC546A -> BC846ASMD; device transistor-npn:TO92-EBC -> transistor-npn:SOT23
- Q4: value BC546A -> BC856ASMD; device transistor-npn:TO92-EBC -> transistor-pnp:SOT23-BEC
- Q6: value BC556 -> BC846ASMD; device transistor-pnp:TO92-EBC -> transistor-npn:SOT23
- moved Q6 57.8 mm to (-80.0, 5.08)
- moved Q5 56.6 mm to (-71.1, 5.08)
- moved Q2 28.5 mm to (-44.5, 5.08)
- moved Q3 28.5 mm to (-53.3, 5.08)
- moved Q4 28.5 mm to (-62.2, 5.08)
- moved Q1 3.81 mm to (-35.6, 5.08)
Changed lines of the file:
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@@
 <?xml version="1.0" encoding="utf-8"?>
 <!DOCTYPE eagle SYSTEM "eagle.dtd">
-<eagle version="6.6.0">
+<eagle version="7.2.0">
 <drawing>
 <settings>
@@
 <layers>
 <layer number="1" name="Top" color="4" fill="1" visible="yes" active="yes"/>
+<layer number="2" name="Route2" color="1" fill="3" visible="no" active="yes"/>
+<layer number="3" name="Route3" color="4" fill="3" visible="no" active="yes"/>
+<layer number="4" name="Route4" color="1" fill="4" visible="no" active="yes"/>
+<layer number="5" name="Route5" color="4" fill="4" visible="no" active="yes"/>
+<layer number="6" name="Route6" color="1" fill="8" visible="no" active="yes"/>
+<layer number="7" name="Route7" color="4" fill="8" visible="no" active="yes"/>
+<layer number="8" name="Route8" color="1" fill="2" visible="no" active="yes"/>
+<layer number="9" name="Route9" color="4" fill="2" visible="no" active="yes"/>
+<layer number="10" name="Route10" color="1" fill="7" visible="no" active="yes"/>
+<layer number="11" name="Route11" color="4" fill="7" visible="no" active="yes"/>
+<layer number="12" name="Route12" color="1" fill="5" visible="no" active="yes"/>
+<layer number="13" name="Route13" color="4" fill="5" visible="no" active="yes"/>
+<layer number="14" name="Route14" color="1" fill="6" visible="no" active="yes"/>
+<layer number="15" name="Route15" color="4" fill="6" visible="no" active="yes"/>
 <layer number="16" name="Bottom" color="1" fill="1" visible="yes" active="yes"/>
 <layer number="17" name="Pads" color="2" fill="1" visible="yes" active="yes"/>
@@
 <pass name="Default">
 <param name="RoutingGrid" value="50mil"/>
+<param name="AutoGrid" value="1"/>
+<param name="Efforts" value="0"/>
+<param name="TopRouterVariant" value="1"/>
 <param name="tpViaShape" value="round"/>
 <param name="PrefDir.1" value="|"/>
@@
 </autorouter>
 <elements>
-<element name="IC1" library="linear" package="DIL08" value="TL072P" x="44.45" y="31.75" rot="R270"/>
-<element name="Q1" library="transistor-npn" package="TO92-EBC" value="BC546A" x="-31.75" y="5.08"/>
-<element name="Q2" library="transistor-npn" package="TO92-EBC" value="BC546A" x="-17.78" y="15.24"/>
-<element name="Q3" library="transistor-npn" package="TO92-EBC" value="BC546A" x="-26.67" y="15.24"/>
-<element name="Q4" library="transistor-npn" package="TO92-EBC" value="BC546A" x="-35.56" y="15.24"/>
-<element name="Q5" library="transistor-npn" package="TO92-EBC" value="BC546A" x="-17.78" y="24.13"/>
-<element name="Q6" library="transistor-pnp" package="TO92-EBC" value="BC556" x="-25.4" y="24.13"/>
+<element name="IC1" library="linear" package="SO08" value="TL072D" x="44.45" y="31.75" rot="R270"/>
 <element name="D1" library="diode" package="DO35-7" value="1N4148DO35-7" x="-24.13" y="31.75"/>
+<element name="Q1" library="transistor-npn" package="SOT23" value="BC846ASMD" x="-35.56" y="5.08"/>
+<element name="Q2" library="transistor-npn" package="SOT23" value="BC846ASMD" x="-44.45" y="5.08"/>
+<element name="Q3" library="transistor-npn" package="SOT23" value="BC846ASMD" x="-53.34" y="5.08"/>
+<element name="Q4" library="transistor-pnp" package="SOT23-BEC" value="BC856ASMD" x="-62.23" y="5.08"/>
+<element name="Q5" library="transistor-npn" package="SOT23" value="BC846ASMD" x="-71.12" y="5.08"/>
+<element name="Q6" library="transistor-npn" package="SOT23" value="BC846ASMD" x="-80.01" y="5.08"/>
+<element name="D2" library="diode" package="DO35-7" value="1N4148DO35-7" x="-77.47" y="-3.81"/>
+<element name="D3" library="diode" package="DO35-7" value="1N4148DO35-7" x="-77.47" y="-10.16"/>
+<element name="C1" library="capacitor-wima" package="C2.5-2" value="" x="-80.01" y="-17.78"/>
+<element name="C2" library="rcl" package="E2-5" value="" x="-80.01" y="-22.86"/>
+<element name="C3" library="rcl" package="E2-5" value="" x="-80.01" y="-29.21"/>
+<element name="C4" library="rcl" package="E2-5" value="" x="-80.01" y="-35.56"/>
+<element name="C5" library="rcl" package="E2-5" value="" x="-80.01" y="-41.91"/>
+<element name="C6" library="rcl" package="E2-5" value="" x="-80.01" y="-48.26"/>
+<element name="C7" library="rcl" package="E2-5" value="" x="-80.01" y="-54.61"/>
+<element name="C8" library="capacitor-wima" package="C2.5-2" value="" x="-80.01" y="-60.96"/>
+<element name="C9" library="capacitor-wima" package="C2.5-2" value="" x="-80.01" y="-66.04"/>
+<element name="C10" library="capacitor-wima" package="C2.5-2" value="" x="-80.01" y="-71.12"/>
+<element name="C11" library="capacitor-wima" package="C2.5-2" value="" x="-80.01" y="-76.2"/>
+<element name="C12" library="capacitor-wima" package="C2.5-2" value="" x="-80.01" y="-81.28"/>
+<element name="C13" library="capacitor-wima" package="C2.5-2" value="" x="-80.01" y="-86.36"/>
+<element name="C14" library="capacitor-wima" package="C2.5-2" value="" x="-80.01" y="-91.44"/>
 </elements>
 <signals>
