File: 808_Kick.brd (EAGLE design)
At the start: 55.6 x 36.8 mm, 58 parts, among them IC1 TL072P, Q1 BC546A, Q2 BC546A, Q3 BC546A, Q4 BC546A, Q5 BC546A, Q6 BC556

Commit message: Board Completed
Board Complete - Gerber files generated
Parts:
- moved R10 2.12 mm to (19.9, 4.31)
- moved R3 1.84 mm to (25.8, 4.31)
- moved R23 1.80 mm to (33.3, 4.31)
- moved D3 1.56 mm to (5.25, 3.72)
- moved R19 0.67 mm to (16.9, 15.4)
- moved R12 0.60 mm to (12.4, 16.2)
- moved _-__G_+_ 0.24 mm to (2.60, 26.4)
Routing:
- net GND: track 0.00 -> 161.4 mm
- net -15V: track 0.00 -> 73.2 mm
- net +15V: track 0.00 -> 69.1 mm
- net N$25: track 0.00 -> 37.4 mm
- net N$12: track 0.00 -> 37.3 mm
- net N$10: track 0.00 -> 32.0 mm
- net FREQ: track 0.00 -> 30.0 mm
- net N$18: track 0.00 -> 28.7 mm
- net N$14: track 0.00 -> 25.8 mm
- net N$9: track 0.00 -> 24.6 mm
- net N$32: track 0.00 -> 23.9 mm
- net N$4: track 0.00 -> 23.1 mm
- net N$28: track 0.00 -> 21.8 mm
- net N$2: track 0.00 -> 21.1 mm
- net N$19: track 0.00 -> 21.0 mm
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