File: 808_Kick.sch (EAGLE design)
At the start: 8 parts, among them IC1 TL072P, Q1 BC546A, Q2 BC546A, Q3 BC546A, Q4 BC546A, Q5 BC546A, Q6 BC556

Commit message: Updated
Parts:
- added C1, C10, C11, C12, C13, C14, C8, C9: (no value), capacitor-wima:C2.5/2
- added C2, C3, C4, C5, C6, C7: (no value), rcl:CPOL-USE2-5
- added D2, D3: 1N4148DO35-7, diode:1N4148DO35-7
- IC1: value TL072P -> TL072D; device linear:TL072P -> linear:TL072D
- Q1, Q2, Q3, Q5: value BC546A -> BC846ASMD; device transistor-npn:BC546A -> transistor-npn:BC846ASMD
- Q4: value BC546A -> BC856ASMD; device transistor-npn:BC546A -> transistor-pnp:BC856ASMD
- Q6: value BC556 -> BC846ASMD; device transistor-pnp:BC556 -> transistor-npn:BC846ASMD
Other:
- moved on the sheet: D1, IC1A, IC1B, Q1, Q2, Q3, Q5
Changed lines of the file:
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@@
 <?xml version="1.0" encoding="utf-8"?>
 <!DOCTYPE eagle SYSTEM "eagle.dtd">
-<eagle version="6.6.0">
+<eagle version="7.2.0">
 <drawing>
 <settings>
@@
 <layers>
 <layer number="1" name="Top" color="4" fill="1" visible="no" active="no"/>
+<layer number="2" name="Route2" color="1" fill="3" visible="no" active="no"/>
+<layer number="3" name="Route3" color="4" fill="3" visible="no" active="no"/>
+<layer number="4" name="Route4" color="1" fill="4" visible="no" active="no"/>
+<layer number="5" name="Route5" color="4" fill="4" visible="no" active="no"/>
+<layer number="6" name="Route6" color="1" fill="8" visible="no" active="no"/>
+<layer number="7" name="Route7" color="4" fill="8" visible="no" active="no"/>
+<layer number="8" name="Route8" color="1" fill="2" visible="no" active="no"/>
+<layer number="9" name="Route9" color="4" fill="2" visible="no" active="no"/>
+<layer number="10" name="Route10" color="1" fill="7" visible="no" active="no"/>
+<layer number="11" name="Route11" color="4" fill="7" visible="no" active="no"/>
+<layer number="12" name="Route12" color="1" fill="5" visible="no" active="no"/>
+<layer number="13" name="Route13" color="4" fill="5" visible="no" active="no"/>
+<layer number="14" name="Route14" color="1" fill="6" visible="no" active="no"/>
+<layer number="15" name="Route15" color="4" fill="6" visible="no" active="no"/>
 <layer number="16" name="Bottom" color="1" fill="1" visible="no" active="no"/>
 <layer number="17" name="Pads" color="2" fill="1" visible="no" active="no"/>
@@
 </classes>
 <parts>
-<part name="IC1" library="linear" deviceset="TL072" device="P"/>
-<part name="Q1" library="transistor-npn" deviceset="BC546*" device="" technology="A"/>
-<part name="Q2" library="transistor-npn" deviceset="BC546*" device="" technology="A"/>
-<part name="Q3" library="transistor-npn" deviceset="BC546*" device="" technology="A"/>
-<part name="Q4" library="transistor-npn" deviceset="BC546*" device="" technology="A"/>
-<part name="Q5" library="transistor-npn" deviceset="BC546*" device="" technology="A"/>
-<part name="Q6" library="transistor-pnp" deviceset="BC556*" device=""/>
+<part name="IC1" library="linear" deviceset="TL072" device="D" value="TL072D"/>
 <part name="D1" library="diode" deviceset="1N4148" device="DO35-7"/>
+<part name="Q1" library="transistor-npn" deviceset="BC846*" device="SMD" technology="A"/>
+<part name="Q2" library="transistor-npn" deviceset="BC846*" device="SMD" technology="A"/>
+<part name="Q3" library="transistor-npn" deviceset="BC846*" device="SMD" technology="A"/>
+<part name="Q4" library="transistor-pnp" deviceset="BC856*" device="SMD" technology="A"/>
+<part name="Q5" library="transistor-npn" deviceset="BC846*" device="SMD" technology="A"/>
+<part name="Q6" library="transistor-npn" deviceset="BC846*" device="SMD" technology="A"/>
+<part name="D2" library="diode" deviceset="1N4148" device="DO35-7"/>
+<part name="D3" library="diode" deviceset="1N4148" device="DO35-7"/>
+<part name="C1" library="capacitor-wima" deviceset="C" device="2.5/2"/>
+<part name="C2" library="rcl" deviceset="CPOL-US" device="E2-5"/>
+<part name="C3" library="rcl" deviceset="CPOL-US" device="E2-5"/>
+<part name="C4" library="rcl" deviceset="CPOL-US" device="E2-5"/>
+<part name="C5" library="rcl" deviceset="CPOL-US" device="E2-5"/>
+<part name="C6" library="rcl" deviceset="CPOL-US" device="E2-5"/>
+<part name="C7" library="rcl" deviceset="CPOL-US" device="E2-5"/>
+<part name="C8" library="capacitor-wima" deviceset="C" device="2.5/2"/>
+<part name="C9" library="capacitor-wima" deviceset="C" device="2.5/2"/>
+<part name="C10" library="capacitor-wima" deviceset="C" device="2.5/2"/>
+<part name="C11" library="capacitor-wima" deviceset="C" device="2.5/2"/>
+<part name="C12" library="capacitor-wima" deviceset="C" device="2.5/2"/>
+<part name="C13" library="capacitor-wima" deviceset="C" device="2.5/2"/>
+<part name="C14" library="capacitor-wima" deviceset="C" device="2.5/2"/>
 </parts>
 <sheets>
@@
 </plain>
 <instances>
-<instance part="IC1" gate="A" x="45.72" y="66.04"/>
-<instance part="IC1" gate="B" x="96.52" y="99.06"/>
-<instance part="Q1" gate="G$1" x="2.54" y="58.42"/>
-<instance part="Q2" gate="G$1" x="40.64" y="91.44"/>
-<instance part="Q3" gate="G$1" x="40.64" y="134.62"/>
-<instance part="Q4" gate="G$1" x="22.86" y="134.62"/>
-<instance part="Q5" gate="G$1" x="142.24" y="68.58"/>
-<instance part="Q6" gate="G$1" x="7.62" y="76.2"/>
-<instance part="D1" gate="G$1" x="30.48" y="58.42" rot="R90"/>
+<instance part="IC1" gate="A" x="45.72" y="63.5" rot="MR180"/>
+<instance part="IC1" gate="B" x="99.06" y="99.06" rot="MR180"/>
+<instance part="D1" gate="G$1" x="7.62" y="162.56" rot="R270"/>
+<instance part="Q1" gate="G$1" x="-15.24" y="149.86"/>
+<instance part="Q2" gate="G$1" x="-33.02" y="137.16"/>
+<instance part="Q3" gate="G$1" x="40.64" y="91.44"/>
+<instance part="Q4" gate="G$1" x="2.54" y="73.66"/>
+<instance part="Q5" gate="G$1" x="-2.54" y="55.88"/>
+<instance part="Q6" gate="G$1" x="127" y="55.88"/>
+<instance part="D2" gate="G$1" x="27.94" y="55.88" rot="R90"/>
+<instance part="D3" gate="G$1" x="-40.64" y="78.74"/>
+<instance part="C1" gate="G$1" x="-27.94" y="78.74" rot="R90"/>
+<instance part="C2" gate="G$1" x="83.82" y="71.12" rot="R270"/>
+<instance part="C3" gate="G$1" x="160.02" y="144.78" rot="R180"/>
+<instance part="C4" gate="G$1" x="91.44" y="177.8"/>
+<instance part="C5" gate="G$1" x="101.6" y="55.88" rot="R90"/>
+<instance part="C6" gate="G$1" x="93.98" y="121.92" rot="R90"/>
+<instance part="C7" gate="G$1" x="91.44" y="190.5"/>
+<instance part="C8" gate="G$1" x="-25.4" y="147.32"/>
+<instance part="C9" gate="G$1" x="53.34" y="104.14" rot="R90"/>
+<instance part="C10" gate="G$1" x="73.66" y="66.04" rot="R180"/>
+<instance part="C11" gate="G$1" x="66.04" y="104.14" rot="R270"/>
+<instance part="C12" gate="G$1" x="-2.54" y="167.64" rot="R90"/>
+<instance part="C13" gate="G$1" x="139.7" y="45.72"/>
+<instance part="C14" gate="G$1" x="17.78" y="66.04" rot="R90"/>
 </instances>
 <busses>
